Commit message: Add base links to all urdfs

File: planar_leg_linkage.urdf (robot description, URDF)
Before this commit: robot planar_leg_linkage, 4 links, 3 joints
Links:
- added link base
Joints:
- added joint base_to_thigh: type continuous, parent base, child thigh, origin xyz=0.0 0.0 0.0, axis 0 0 1

File: revolute_rotor_chain.urdf (robot description, URDF)
Before this commit: robot revolute_rotor_chain, 7 links, 6 joints
Links:
- removed link base_link
- removed link link1
- removed link link2
- removed link link3
- removed link rotor1
- removed link rotor2
- removed link rotor3
- added link ground
- added link link-0, mass 1
- added link link-1, mass 1
- added link link-2, mass 1
- added link rotor-0, mass 1
- added link rotor-1, mass 1
- added link rotor-2, mass 1
Joints:
- joint joint1: child link1 -> link-0; parent base_link -> ground
- joint joint1r: child rotor1 -> rotor-0; parent base_link -> ground
- joint joint2: child link2 -> link-1; parent link1 -> link-0
- joint joint2r: child rotor2 -> rotor-1; parent link1 -> link-0
- joint joint3: child link3 -> link-2; parent link2 -> link-1
- joint joint3r: child rotor3 -> rotor-2; parent link2 -> link-1
