Commit message: - Add inertia to rev chain urdf - Add constraint joints to rev rotor chain urdf - Remove axis element from all constraint joints

File: revolute_rotor_chain.urdf (robot description, URDF)
Before this commit: robot revolute_rotor_chain, 7 links, 6 joints
Links:
- link link1: mass None -> 1
- link link2: mass None -> 1
- link link3: mass None -> 1
- link rotor1: mass None -> 1
- link rotor2: mass None -> 1
- link rotor3: mass None -> 1

Commit message: Rev with rotor chain agrees with manual model

File: revolute_rotor_chain.urdf (robot description, URDF)
Before this commit: robot revolute_rotor_chain, 7 links, 6 joints
Links:
- link rotor-0: mass 1 -> 0
- link rotor-1: mass 1 -> 0
- link rotor-2: mass 1 -> 0
Joints:
- joint joint2: origin (none) -> xyz=1.0 0.0 0.0
- joint joint2r: origin (none) -> xyz=1.0 0.0 0.0
- joint joint3: origin (none) -> xyz=1.0 0.0 0.0
- joint joint3r: origin (none) -> xyz=1.0 0.0 0.0
