Commit message: WIP mini cheetah urdf

File: mini_cheetah.urdf (robot description, URDF)
Before this commit: robot mini_cheetah, 25 links, 24 joints
Links:
- link abduct_rotor_fr: mass 0.054 -> 0.
Joints:
- joint torso_to_abduct_fr_j: origin xyz=0.19 -0.049 0.0 rpy=0 0 0 -> xyz=0.19 -0.05 0.0 rpy=0 0 0

Commit message: Build mini cheetah urdf using xacro

File: mini_cheetah.urdf (robot description, URDF)
Before this commit: robot mini_cheetah, 25 links, 24 joints
Links:
- removed link abduct_fl
- removed link abduct_fr
- removed link abduct_hl
- removed link abduct_hr
- removed link abduct_rotor_fl
- removed link abduct_rotor_fr
- removed link abduct_rotor_hl
- removed link abduct_rotor_hr
- removed link body
- removed link hip_rotor_fl
- removed link hip_rotor_fr
- removed link hip_rotor_hl
- removed link hip_rotor_hr
- removed link knee_rotor_fl
- removed link knee_rotor_fr
- removed link knee_rotor_hl
- removed link knee_rotor_hr
- removed link shank_fl
- removed link shank_fr
- removed link shank_hl
- removed link shank_hr
- removed link thigh_fl
- removed link thigh_fr
- removed link thigh_hl
- removed link thigh_hr
- added link FL_abad_link, mass 0.54
- added link FL_abad_rotor, mass 0.
- added link FL_hip_link, mass 0.634
- added link FL_hip_rotor, mass 0.
- added link FL_knee_link, mass 0.064
- added link FL_knee_rotor, mass 0.
- added link FR_abad_link, mass 0.54
- added link FR_abad_rotor, mass 0.
- added link FR_hip_link, mass 0.634
- added link FR_hip_rotor, mass 0.
- added link FR_knee_link, mass 0.064
- added link FR_knee_rotor, mass 0.
- added link Floating Base, mass 3.3
- added link HL_abad_link, mass 0.54
- added link HL_abad_rotor, mass 0.
- added link HL_hip_link, mass 0.634
- added link HL_hip_rotor, mass 0.
- added link HL_knee_link, mass 0.064
- added link HL_knee_rotor, mass 0.
- added link HR_abad_link, mass 0.54
- added link HR_abad_rotor, mass 0.
- added link HR_hip_link, mass 0.634
- added link HR_hip_rotor, mass 0.
- added link HR_knee_link, mass 0.064
- added link HR_knee_rotor, mass 0.
Joints:
- removed joint abduct_fl_to_hip_rotor_fl_j
- removed joint abduct_fl_to_thigh_fl_j
- removed joint abduct_fr_to_hip_rotor_fr_j
- removed joint abduct_fr_to_thigh_fr_j
- removed joint abduct_hl_to_hip_rotor_hl_j
- removed joint abduct_hl_to_thigh_hl_j
- removed joint abduct_hr_to_hip_rotor_hr_j
- removed joint abduct_hr_to_thigh_hr_j
- removed joint hip_fl_to_knee_rotor_fl_j
- removed joint hip_hl_to_knee_rotor_hl_j
- removed joint hip_hr_to_knee_rotor_hr_j
- removed joint hip_rotor_fr_to_knee_rotor_fr_j
- removed joint thigh_fl_to_knee_fl_j
- removed joint thigh_fr_to_knee_fr_j
- removed joint thigh_hl_to_knee_hl_j
- removed joint thigh_hr_to_knee_hr_j
- removed joint torso_to_abduct_fl_j
- removed joint torso_to_abduct_fr_j
- removed joint torso_to_abduct_hl_j
- removed joint torso_to_abduct_hr_j
- removed joint torso_to_abduct_rotor_fl_j
- removed joint torso_to_abduct_rotor_fr_j
- removed joint torso_to_abduct_rotor_hl_j
- removed joint torso_to_abduct_rotor_hr_j
- added joint FL_abad_to_hip_j: type continuous, parent FL_abad_link, child FL_hip_link, origin xyz=0 0.062 0.0, axis 0 1 0
- added joint FL_abad_to_hip_rotor_j: type continuous, parent FL_abad_link, child FL_hip_rotor, origin xyz=0.0 0.04 0.0 rpy=0 0 0, axis 0 1 0
- added joint FL_hip_to_knee_j: type continuous, parent FL_hip_link, child FL_knee_link, origin xyz=0.0 0.0 -0.209, axis 0 1 0
- added joint FL_hip_to_knee_rotor_j: type continuous, parent FL_hip_link, child FL_knee_rotor, axis 0 1 0
- added joint FR_abad_to_hip_j: type continuous, parent FR_abad_link, child FR_hip_link, origin xyz=0 -0.062 0.0, axis 0 1 0
- added joint FR_abad_to_hip_rotor_j: type continuous, parent FR_abad_link, child FR_hip_rotor, origin xyz=0.0 -0.04 0.0 rpy=0 0 0, axis 0 1 0
- added joint FR_hip_to_knee_j: type continuous, parent FR_hip_link, child FR_knee_link, origin xyz=0.0 0.0 -0.209, axis 0 1 0
- added joint FR_hip_to_knee_rotor_j: type continuous, parent FR_hip_link, child FR_knee_rotor, axis 0 1 0
- added joint HL_abad_to_hip_j: type continuous, parent HL_abad_link, child HL_hip_link, origin xyz=0 0.062 0.0, axis 0 1 0
- added joint HL_abad_to_hip_rotor_j: type continuous, parent HL_abad_link, child HL_hip_rotor, origin xyz=0.0 0.04 0.0 rpy=0 0 0, axis 0 1 0
- added joint HL_hip_to_knee_j: type continuous, parent HL_hip_link, child HL_knee_link, origin xyz=0.0 0.0 -0.209, axis 0 1 0
- added joint HL_hip_to_knee_rotor_j: type continuous, parent HL_hip_link, child HL_knee_rotor, axis 0 1 0
- added joint HR_abad_to_hip_j: type continuous, parent HR_abad_link, child HR_hip_link, origin xyz=0 -0.062 0.0, axis 0 1 0
- added joint HR_abad_to_hip_rotor_j: type continuous, parent HR_abad_link, child HR_hip_rotor, origin xyz=0.0 -0.04 0.0 rpy=0 0 0, axis 0 1 0
- added joint HR_hip_to_knee_j: type continuous, parent HR_hip_link, child HR_knee_link, origin xyz=0.0 0.0 -0.209, axis 0 1 0
- added joint HR_hip_to_knee_rotor_j: type continuous, parent HR_hip_link, child HR_knee_rotor, axis 0 1 0
- added joint torso_to_FL_abad_j: type continuous, parent Floating Base, child FL_abad_link, origin xyz=0.19 0.05 0.0, axis 1 0 0
- added joint torso_to_FL_abad_rotor_j: type continuous, parent Floating Base, child FL_abad_rotor, origin xyz=0.125 0.049 0.0, axis 1 0 0
- added joint torso_to_FR_abad_j: type continuous, parent Floating Base, child FR_abad_link, origin xyz=0.19 -0.05 0.0, axis 1 0 0
- added joint torso_to_FR_abad_rotor_j: type continuous, parent Floating Base, child FR_abad_rotor, origin xyz=0.125 -0.049 0.0, axis 1 0 0
- added joint torso_to_HL_abad_j: type continuous, parent Floating Base, child HL_abad_link, origin xyz=-0.19 0.05 0.0, axis 1 0 0
- added joint torso_to_HL_abad_rotor_j: type continuous, parent Floating Base, child HL_abad_rotor, origin xyz=-0.125 0.049 0.0, axis 1 0 0
- added joint torso_to_HR_abad_j: type continuous, parent Floating Base, child HR_abad_link, origin xyz=-0.19 -0.05 0.0, axis 1 0 0
- added joint torso_to_HR_abad_rotor_j: type continuous, parent Floating Base, child HR_abad_rotor, origin xyz=-0.125 -0.049 0.0, axis 1 0 0
