Commit message: WIP

File: four_bar.urdf (robot description, URDF)
Before this commit: robot four_bar, 4 links, 3 joints
Links:
- link base_link: mass 3.3 -> None

File: six_bar.urdf (robot description, URDF)
Before this commit: robot six_bar, 6 links, 5 joints
Links:
- link base_link: mass 3.3 -> None
